Commit message: adding changes

File: objects/test_cube1.urdf (robot description, URDF)
Before this commit: robot block, 1 links, 0 joints
Links:
- link block: geometry collision box size=0.5 0.5 0.0001; visual box size=0.5 0.5 0.0001

File: objects/test_cube3.urdf (robot description, URDF)
Before this commit: robot block, 1 links, 0 joints
Links:
- link block: geometry collision box size=0.05 0.05 0.05; visual box size=0.05 0.05 0.05
