Commit message: adding debug function

File: objects/test_cube4.urdf (robot description, URDF)
Before this commit: robot block, 1 links, 0 joints
Links:
- link block: geometry collision box size=0.003 0.003 0.05; visual box size=0.003 0.003 0.05

Commit message: fine tuning conversion rate for pixels

File: objects/test_cube4.urdf (robot description, URDF)
Before this commit: robot block, 1 links, 0 joints
Links:
- link block: geometry collision box size=0.001 0.001 0.05; visual box size=0.0001 0.0001 0.05

Commit message: fixing img width bug

File: objects/test_cube4.urdf (robot description, URDF)
Before this commit: robot block, 1 links, 0 joints
Links:
- link block: geometry collision box size=0.005 0.005 0.05; visual box size=0.002 0.002 0.05

Commit message: adding object wrapper

File: objects/test_cube4.urdf (robot description, URDF)
Before this commit: robot block, 1 links, 0 joints
Links:
- link block: geometry collision box size=0.005 0.005 0.05; visual box size=0.001 0.001 0.05
